File: hardware/KiCad/mini-MCU-LINK-Integrated/mini-MCU-LINK-Integrated.kicad_pcb (KiCad board)
At the start: 2 copper layers, 57 parts, among them J1 USB4110-GF-A_REVB, J2 BM03B-SRSS-TB, J3 Conn_02x05_Odd_Even, Q1 PMDXB290UNE, Q2 PMDXB290UNE, Q3 PMDXB290UNE, Q4 PMDXB290UNE, SW1 KMR221GLFS, U1 XC6227C331PR-G, U2 LPC55S69JBD64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

Commit message: added notes, updated 3D model
Other:
- board text removed: "Mit Stecker"
- board text removed: "Ohne Stecker"
Changed lines of the file:
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@@
     (effects (font (size 0.8 0.8) (thickness 0.15)) (justify left bottom))
-  )
-  (gr_text "Ohne Stecker " (at 98.7 94.2) (layer "F.SilkS")
-    (effects (font (size 1 1) (thickness 0.15)) (justify left bottom))
-  )
-  (gr_text "Mit Stecker" (at 104.1 68.6) (layer "F.SilkS")
-    (effects (font (size 1 1) (thickness 0.15)) (justify left bottom))
   )
   (gr_text "Firmware" (at 103.29006 73.331492) (layer "F.SilkS")
@@
     (polygon
       (pts
-        (xy 95.1 63.9)
+        (xy 95.4302 65.8304)
         (xy 95.1 98.5)
         (xy 148.3 98)
-        (xy 148 64.1)
+        (xy 148.3302 66.0304)
       )
     )
