File: hardware/KiCad/mini-MCU-Link-Drone/mculink_standalone_debug_uart.kicad_sch (KiCad schematic)
At the start: 23 parts, among them J2 BM03B-SRSS-TB, J3 Conn_02x05_Odd_Even, J4 Conn_01x10_Pin, J5 Conn_01x06_Pin, Q1 PMDXB290UNE, Q2 PMDXB290UNE, Q3 PMDXB290UNE, SW1 KMR221GLFS, SW2 KMR221GLFS, U2 LPC55S69JBD64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

Commit message: updated schematic part
Connections:
- net GND: now also J4.10 (Pin_10), J5.6 (Pin_6)
- no-connect marks 28 -> 42
Changed lines of the file:
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@@
   )
   (no_connect (at 215.9 55.88))
+  (no_connect (at 267.97 127))
   (no_connect (at 34.29 48.26))
   (no_connect (at 33.02 123.19))
   (no_connect (at 34.29 86.36))
+  (no_connect (at 234.95 130.81))
   (no_connect (at 33.02 120.65))
   (no_connect (at 82.55 140.97))
   (no_connect (at 87.63 133.35))
   (no_connect (at 34.29 45.72))
+  (no_connect (at 234.95 118.11))
   (no_connect (at 34.29 99.06))
   (no_connect (at 77.47 133.35))
+  (no_connect (at 234.95 125.73))
   (no_connect (at 34.29 101.6))
   (no_connect (at 34.29 53.34))
@@
   (no_connect (at 203.2 63.5))
   (no_connect (at 34.29 66.04))
+  (no_connect (at 234.95 123.19))
   (no_connect (at 34.29 60.96))
+  (no_connect (at 234.95 120.65))
   (no_connect (at 34.29 104.14))
+  (no_connect (at 234.95 135.89))
+  (no_connect (at 234.95 138.43))
   (no_connect (at 34.29 81.28))
+  (no_connect (at 267.97 124.46))
+  (no_connect (at 267.97 132.08))
+  (no_connect (at 267.97 129.54))
+  (no_connect (at 267.97 134.62))
   (no_connect (at 34.29 78.74))
   (no_connect (at 34.29 68.58))
   (no_connect (at 34.29 73.66))
+  (no_connect (at 234.95 133.35))
   (no_connect (at 34.29 93.98))
   (no_connect (at 34.29 71.12))
   (no_connect (at 34.29 43.18))
+  (no_connect (at 234.95 128.27))
   (no_connect (at 34.29 38.1))
   (no_connect (at 33.02 125.73))
@@
     (stroke (width 0) (type default))
   )
+  (wire (pts (xy 236.22 140.97) (xy 236.22 142.24))
+    (stroke (width 0) (type default))
+  )
+  (wire (pts (xy 267.97 137.16) (xy 269.24 137.16))
+    (stroke (width 0) (type default))
+  )
   (wire (pts (xy 71.12 166.37) (xy 71.12 170.18))
     (stroke (width 0) (type default))
@@
     (stroke (width 0) (type default))
   )
+  (wire (pts (xy 269.24 137.16) (xy 269.24 139.7))
+    (stroke (width 0) (type default))
+  )
   (wire (pts (xy 80.01 45.72) (xy 92.71 45.72))
     (stroke (width 0) (type default))
@@
   )
   (wire (pts (xy 80.01 95.25) (xy 92.71 95.25))
+    (stroke (width 0) (type default))
+  )
+  (wire (pts (xy 234.95 140.97) (xy 236.22 140.97))
     (stroke (width 0) (type default))
   )
@@
     )
   )
+  (symbol (lib_id "power:GND") (at 236.22 142.24 0) (unit 1)
+    (in_bom yes) (on_board yes) (dnp no)
+    (property "Reference" "#PWR063" (at 236.22 148.59 0)
+      (effects (font (size 1.27 1.27)) hide)
+    )
+    (property "Value" "GND" (at 236.347 146.6342 0)
+      (effects (font (size 1.27 1.27)))
+    )
+    (property "Footprint" "" (at 236.22 142.24 0)
+      (effects (font (size 1.27 1.27)) hide)
+    )
+    (property "Datasheet" "" (at 236.22 142.24 0)
+      (effects (font (size 1.27 1.27)) hide)
+    )
+    (pin "1")
+    (instances
+      (project "MCU-Link-Drone"
+        (path "/52afa5f9-012e-424b-bf0c-786f4ecc122a/3cbe4489-d8a9-40e8-8d89-b185e2a351a5"
+          (reference "#PWR063") (unit 1)
+        )
+      )
+      (project "mculink_kicad"
+        (path "/5d025764-753a-4b80-8d3d-c9a8a22c9527/00000000-0000-0000-0000-0000603cfdf2"
+          (reference "#PWR?") (unit 1)
+        )
+      )
+    )
+  )
   (symbol (lib_id "power:GND") (at 158.75 88.9 0) (unit 1)
     (in_bom yes) (on_board yes) (dnp no)
@@
         )
       )
+      (project "mculink_kicad"
+        (path "/5d025764-753a-4b80-8d3d-c9a8a22c9527/00000000-0000-0000-0000-0000603cfdf2"
+          (reference "#PWR?") (unit 1)
+        )
+      )
+    )
+  )
+  (symbol (lib_id "power:GND") (at 269.24 139.7 0) (unit 1)
+    (in_bom yes) (on_board yes) (dnp no)
+    (property "Reference" "#PWR064" (at 269.24 146.05 0)
+      (effects (font (size 1.27 1.27)) hide)
+    )
+    (property "Value" "GND" (at 269.367 144.0942 0)
+      (effects (font (size 1.27 1.27)))
+    )
+    (property "Footprint" "" (at 269.24 139.7 0)
+      (effects (font (size 1.27 1.27)) hide)
+    )
+    (property "Datasheet" "" (at 269.24 139.7 0)
+      (effects (font (size 1.27 1.27)) hide)
+    )
+    (pin "1")
+    (instances
+      (project "MCU-Link-Drone"
+        (path "/52afa5f9-012e-424b-bf0c-786f4ecc122a/3cbe4489-d8a9-40e8-8d89-b185e2a351a5"
+          (reference "#PWR064") (unit 1)
+        )
+      )

Commit message: cleanup and ERC fixes
Parts:
- J2: footprint mculink:JST_BM03B-SRSS-TB_LF__SN_ -> BM03B-SRSS-TB_LF__SN_:JST_BM03B-SRSS-TB_LF__SN_
- Q1, Q2, Q3: footprint mculink:SOT1216 -> Package_TO_SOT_SMD:SOT-363_SC-70-6
- SW1, SW2: symbol mculink_kicad:KMR221GLFS -> mcuoneclipse:KMR221GLFS
- U2: symbol mculink_kicad:LPC55S69JBD64 -> mcuoneclipse:LPC55S69JBD64_PIO0
- U2: symbol mculink_kicad:LPC55S69JBD64 -> mcuoneclipse:LPC55S69JBD64_PIO1
- U3: footprint mculink:SOT95P280X145-5N -> STMPS2141STR:SOT95P280X145-5N
Connections:
- net +3V3: now also U3.4 (EN); no longer U3.5 (IN)
- net GND: now also U3.5 (IN); no longer D2.2 (A), D2.2 (A), D2.2 (A), D2.2 (A), D5.2 (A), D5.2 (A), D5.2 (A), D5.2 (A), U3.4 (EN)

Commit message: made it warning free with KiCAD 8
Parts:
- added R12, R13: 10, Resistor_SMD:R_0402_1005Metric, symbol Device:R
- U2: symbol mcuoneclipse:LPC55S69JBD64_PIO0 -> mcuoneclipse:LPC55S69JBD64
- U2: symbol mcuoneclipse:LPC55S69JBD64_PIO1 -> mcuoneclipse:LPC55S69JBD64
Connections:
- net +3V3: now also R12.2; no longer U2.15 (PIO0_31)
- net GND: now also R13.2; no longer U2.37 (PIO0_9)
- new net: R12.1, U2.15 (PIO0_31)
- new net: R13.1, U2.37 (PIO0_9)
Other:
- note added: "unplaced unit"
- moved on the sheet: D3, R6
