File: hardware/KiCad/mini-MCU-LINK-Standalone/MCU-Link-Standalone.kicad_sch (KiCad schematic)
At the start: 5 parts

Commit message: added notes, updated 3D model
Other:
- note added: "Todo for final v2.2 version: - move ESD protection diodes closer to the pins - check/swap UART header pins to match RPi debug probe cable - Fix DRC errors and warnings"
Changed lines of the file:
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@@
     )
+  )
+  (text "Todo for final v2.2 version:\n- move ESD protection diodes closer to the pins\n- check/swap UART header pins to match RPi debug probe cable\n- Fix DRC errors and warnings\n"
+    (at 182.88 127 0)
+    (effects (font (size 1.27 1.27)) (justify left bottom))
   )
   (symbol (lib_id "power:GND") (at 73.66 127 0) (unit 1)
