File: hardware/KiCad/MCU-Link-Drone/mculink_kicad.kicad_sch (KiCad schematic)
At the start: 7 parts

Commit message: worked on layout
Parts:
- FID1, FID2, FID3: footprint mculink_kicad:Fiducial_1mm_Dia_2.54mm_Outer_CopperTop -> McuOnEclipse:Fiducial_1mm_Dia_2.54mm_Outer_CopperTop; now left out of the parts list
- H1, H2, H3, H4: now left out of the parts list
Changed lines of the file:
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@@
 		(unit 1)
 		(exclude_from_sim no)
-		(in_bom yes)
+		(in_bom no)
 		(on_board yes)
 		(dnp no)
@@
 			)
 		)
-		(property "Footprint" "mculink_kicad:Fiducial_1mm_Dia_2.54mm_Outer_CopperTop"
+		(property "Footprint" "McuOnEclipse:Fiducial_1mm_Dia_2.54mm_Outer_CopperTop"
 			(at 33.02 85.09 0)
 			(effects
@@
 			)
 		)
-		(property "Datasheet" "~"
+		(property "Datasheet" ""
 			(at 33.02 85.09 0)
 			(effects
@@
 		(unit 1)
 		(exclude_from_sim no)
-		(in_bom yes)
+		(in_bom no)
 		(on_board yes)
 		(dnp no)
@@
 			)
 		)
-		(property "Datasheet" "~"
+		(property "Datasheet" ""
 			(at 33.02 97.79 0)
 			(effects
@@
 		(unit 1)
 		(exclude_from_sim no)
-		(in_bom yes)
+		(in_bom no)
 		(on_board yes)
 		(dnp no)
@@
 			)
 		)
-		(property "Footprint" "mculink_kicad:Fiducial_1mm_Dia_2.54mm_Outer_CopperTop"
+		(property "Footprint" "McuOnEclipse:Fiducial_1mm_Dia_2.54mm_Outer_CopperTop"
 			(at 45.72 85.09 0)
 			(effects
@@
 			)
 		)
-		(property "Datasheet" "~"
+		(property "Datasheet" ""
 			(at 45.72 85.09 0)
 			(effects
@@
 		(unit 1)
 		(exclude_from_sim no)
-		(in_bom yes)
+		(in_bom no)
 		(on_board yes)
 		(dnp no)
@@
 			)
 		)
-		(property "Footprint" "mculink_kicad:Fiducial_1mm_Dia_2.54mm_Outer_CopperTop"
+		(property "Footprint" "McuOnEclipse:Fiducial_1mm_Dia_2.54mm_Outer_CopperTop"
 			(at 58.42 85.09 0)
 			(effects
@@
 			)
 		)
-		(property "Datasheet" "~"
+		(property "Datasheet" ""
 			(at 58.42 85.09 0)
 			(effects
@@
 		(unit 1)
 		(exclude_from_sim no)
-		(in_bom yes)
+		(in_bom no)
 		(on_board yes)
 		(dnp no)
@@
 			)
 		)
-		(property "Datasheet" "~"
+		(property "Datasheet" ""
 			(at 54.61 97.79 0)
 			(effects
@@
 		(unit 1)
 		(exclude_from_sim no)
-		(in_bom yes)
+		(in_bom no)
 		(on_board yes)
 		(dnp no)
@@
 			)
 		)
-		(property "Datasheet" "~"
+		(property "Datasheet" ""
 			(at 76.2 97.79 0)
 			(effects
@@
 		(unit 1)
 		(exclude_from_sim no)
-		(in_bom yes)
+		(in_bom no)
 		(on_board yes)
 		(dnp no)
@@
 			)
 		)
-		(property "Datasheet" "~"
+		(property "Datasheet" ""
 			(at 97.79 97.79 0)
 			(effects
