File: hardware/KiCad/MCU-Link_MR/MCU-Link_MR.kicad_pcb (KiCad board)
At the start: 2 copper layers, 57.9 x 39.9 mm, 108 parts, among them J1 Pixhawk Debug Full (1x10 JST-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, J11 JST-GH_BM06B, J2 Pixhawk_Debug_Mini (1x06 JST-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, J3 Jumper_2_Open, J4 Jumper_2_Open, J5 Jumper_2_Open, J6 Conn_02x05_Odd_Even, J8 DCD-LZ_Debug (1x07 JST-GHS), J9 USB4110-GF-A_REVB, SW1 KMR221GLFS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

Commit message: cleanup
Parts:
- removed JP1: SolderJumper_2-3_Open, McuOnEclipse:SolderJumper-3_P1.3mm_Open_RoundedPad1.0x1.5mm
- added JP2: SolderJumper_3_Bridged12, McuOnEclipse:SolderJumper-3_P1.3mm_Open_RoundedPad1.0x1.5mm, B.Cu at (197.9, 83.6)
- moved C31 0.14 mm to (203.4, 102.5)
- moved C30 0.14 mm to (200.4, 102.5)
Connections:
- C34 pad 1: Net-(C34-Pad1) -> /Debug interface/VTARGET
- D4 pad 1: Net-(D4A-K1) -> TX_TO_LPC
- D4 pad 3: Net-(D4B-K2) -> RX_FROM_LPC
- J1 pad 2: FC0_TARGET_RXD -> TX_TO_LPC
- J1 pad 3: FCO_TARGET_TXD -> RX_FROM_LPC
- J11 pad 2: Net-(D4A-K1) -> TX_TO_LPC
- J11 pad 3: Net-(D4B-K2) -> RX_FROM_LPC
- J2 pad 2: FC0_TARGET_RXD -> TX_TO_LPC
- J2 pad 3: FCO_TARGET_TXD -> RX_FROM_LPC
- J8 pad 2: FC0_TARGET_RXD -> TX_TO_LPC
- J8 pad 3: FCO_TARGET_TXD -> RX_FROM_LPC
- R15 pad 2: Net-(C34-Pad1) -> /Debug interface/VTARGET
- R16 pad 1: Net-(C34-Pad1) -> /Debug interface/VTARGET
- R26 pad 2: Net-(D4A-K1) -> TX_TO_LPC
- R27 pad 2: Net-(D4B-K2) -> RX_FROM_LPC
Routing:
- net FC0_TARGET_RXD: track 59.7 -> 11.4 mm, vias 2 -> 0
- net RX_FROM_LPC: track 0.00 -> 46.4 mm, vias 0 -> 4
- net TX_TO_LPC: track 0.00 -> 42.8 mm, vias 0 -> 2
- net FCO_TARGET_TXD: track 56.9 -> 15.6 mm, vias 6 -> 2
- net Net-(D4A-K1): track 13.2 -> 0.00 mm
- net Net-(D4B-K2): track 10.3 -> 0.00 mm
- net /Debug interface/VTARGET: track 62.2 -> 65.7 mm, vias 7 -> 5
- net Net-(C34-Pad1): track 2.97 -> 0.00 mm
- net DBGIF_TMS_SWDIO_TXEN: track 18.7 -> 19.4 mm
- net GND: vias 124 -> 143
